File: hw/sch_pcb/ALTIMET02A.kicad_sch (KiCad schematic)
At the start: 14 parts, among them IC1 MS561101BA03-50, J1 HEADER_2x03_PARALLEL, J2 HEADER_2x03, J3 HEADER_2x05_PARALLEL

Commit message: Fix title block.
Other:
- company: (none) -> Marek Sommer
- title: (none) -> ALTIMET02
Changed lines of the file:
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@@
 (kicad_sch (version 20211123) (generator eeschema)
   (paper "A4")
+  (title_block
+    (title "ALTIMET02")
+    (date "2023-01-18")
+    (rev "A")
+    (company "Marek Sommer")
+    (comment 1 "Digital altimeter  \\nand barometer sensor")
+  )
   (junction (at 93.345 76.2) (diameter 0) (color 0 0 0 0)
   )
@@
       (effects (font (size 1.27 1.27)) (justify left) hide)
     )
-    (property "Datasheet" "http://www.te.com/usa-en/search.html?q=ms5611&source=header" (id 3) (at 157.48 76.2 0)
+    (property "Datasheet" "https://www.te.com/usa-en/product-MS561101BA03-50.datasheet.pdf" (id 3) (at 157.48 76.2 0)
       (effects (font (size 1.27 1.27)) (justify left) hide)
     )
