File: hw/sch_pcb/ALTIMET02.kicad_sch (KiCad schematic)
At the start: 17 parts, among them J1 HEADER_2x02_PARALLEL, J2 HEADER_2x03_PARALLEL, J3 HEADER_2x05_PARALLEL, U1 MS5611-01BA

Commit message: add ustid
Parts:
- C1: UST_ID (none) -> 5c70984712875079b91f8b53
- C2: UST_ID (none) -> 5c70984712875079b91f8b4c
- D1: UST_ID (none) -> 650b35ab462c6d9e720543d0
- R1, R2: value 5k -> 5k1; UST_ID (none) -> 5fa0fc3e12875025b3977997
- U1: UST_ID (none) -> 650b36b0462c6d9e720543f4
Changed lines of the file:
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@@
+      (effects (font (size 1.27 1.27)) hide)
+    )
+    (property "UST_ID" "" (at 261.62 48.26 0)
       (effects (font (size 1.27 1.27)) hide)
     )
@@
     )
     (property "Datasheet" "~" (at 147.32 132.08 0)
+      (effects (font (size 1.27 1.27)) hide)
+    )
+    (property "UST_ID" "" (at 147.32 132.08 0)
       (effects (font (size 1.27 1.27)) hide)
     )
@@
     (property "Datasheet" "" (at 251.46 121.92 0)
       (effects (font (size 1.524 1.524)))
+    )
+    (property "UST_ID" "" (at 251.46 127 0)
+      (effects (font (size 1.27 1.27)) hide)
     )
     (pin "1")
@@
       (effects (font (size 1.524 1.524)))
     )
+    (property "UST_ID" "" (at 157.48 38.1 0)
+      (effects (font (size 1.27 1.27)) hide)
+    )
     (pin "1")
     (pin "2")
@@
       (effects (font (size 1.27 1.27)) hide)
     )
+    (property "UST_ID" "650b35ab462c6d9e720543d0" (at 71.12 67.31 0)
+      (effects (font (size 1.27 1.27)) hide)
+    )
     (pin "1")
     (pin "2")
@@
       (effects (font (size 1.27 1.27)) (justify left))
     )
-    (property "Value" "5k" (at 232.41 119.38 0)
+    (property "Value" "5k1" (at 232.41 119.38 0)
       (effects (font (size 1.27 1.27)) (justify left))
     )
@@
     )
     (property "Datasheet" "~" (at 229.87 118.11 0)
+      (effects (font (size 1.27 1.27)) hide)
+    )
+    (property "UST_ID" "5fa0fc3e12875025b3977997" (at 229.87 118.11 0)
       (effects (font (size 1.27 1.27)) hide)
     )
@@
     )
     (property "Datasheet" "~" (at 254 31.75 0)
+      (effects (font (size 1.27 1.27)) hide)
+    )
+    (property "UST_ID" "" (at 254 31.75 0)
       (effects (font (size 1.27 1.27)) hide)
     )
@@
     )
     (property "Datasheet" "https://www.te.com/commerce/DocumentDelivery/DDEController?Action=srchrtrv&DocNm=MS5611-01BA03&DocType=Data+Sheet&DocLang=English" (at 130.81 77.47 0)
+      (effects (font (size 1.27 1.27)) hide)
+    )
+    (property "UST_ID" "650b36b0462c6d9e720543f4" (at 130.81 77.47 0)
       (effects (font (size 1.27 1.27)) hide)
     )
@@
       (effects (font (size 1.524 1.524)))
     )
+    (property "UST_ID" "" (at 251.46 77.47 0)
+      (effects (font (size 1.27 1.27)) hide)
+    )
     (pin "1")
     (pin "2")
@@
       (effects (font (size 1.27 1.27)) hide)
     )
+    (property "UST_ID" "5c70984712875079b91f8b4c" (at 95.25 67.31 0)
+      (effects (font (size 1.27 1.27)) hide)
+    )
     (pin "1")
     (pin "2")
@@
       (effects (font (size 1.27 1.27)) hide)
     )
+    (property "UST_ID" "" (at 261.62 31.75 0)
+      (effects (font (size 1.27 1.27)) hide)
+    )
     (pin "1")
     (instances
@@
     )
     (property "Datasheet" "~" (at 246.38 48.26 0)
+      (effects (font (size 1.27 1.27)) hide)
+    )
+    (property "UST_ID" "" (at 246.38 48.26 0)
       (effects (font (size 1.27 1.27)) hide)
     )
@@
     )
     (property "Datasheet" "~" (at 269.24 31.75 0)
+      (effects (font (size 1.27 1.27)) hide)
+    )
+    (property "UST_ID" "" (at 269.24 31.75 0)
       (effects (font (size 1.27 1.27)) hide)
     )
@@
       (effects (font (size 1.27 1.27)) hide)
     )
+    (property "UST_ID" "" (at 246.38 31.75 0)
+      (effects (font (size 1.27 1.27)) hide)
+    )
     (pin "1")
     (instances
@@
       (effects (font (size 1.27 1.27)) hide)
     )
+    (property "UST_ID" "5c70984712875079b91f8b53" (at 82.55 67.31 0)
+      (effects (font (size 1.27 1.27)) hide)
+    )
     (pin "1")
     (pin "2")
@@
       (effects (font (size 1.27 1.27)) hide)
     )
+    (property "UST_ID" "" (at 116.84 133.35 0)
+      (effects (font (size 1.27 1.27)) hide)
+    )
     (pin "1")
     (pin "2")
@@
       (effects (font (size 1.27 1.27)) (justify left))
     )
-    (property "Value" "5k" (at 222.25 119.38 0)
+    (property "Value" "5k1" (at 222.25 119.38 0)
       (effects (font (size 1.27 1.27)) (justify left))
     )
@@
       (effects (font (size 1.27 1.27)) hide)
     )
+    (property "UST_ID" "5fa0fc3e12875025b3977997" (at 219.71 118.11 0)
+      (effects (font (size 1.27 1.27)) hide)
+    )

Commit message: Upravy a kontrola pred vyrobou
Parts:
- U1: footprint Package_LGA:LGA-8_3x5mm_P1.25mm -> Mlab_IO:MS5611-01BA03
Changed lines of the file:
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@@
       (effects (font (size 1.27 1.27)) (justify left))
     )
-    (property "Footprint" "Package_LGA:LGA-8_3x5mm_P1.25mm" (at 130.81 77.47 0)
+    (property "Footprint" "Mlab_IO:MS5611-01BA03" (at 130.81 77.47 0)
       (effects (font (size 1.27 1.27)) hide)
     )
