File: hw/sch_pcb/ALTIMET02.kicad_pcb (KiCad board)
At the start: 2 copper layers, 40.1 x 19.8 mm, 17 parts, among them J1 HEADER_2x02_PARALLEL, J2 HEADER_2x03_PARALLEL, J3 HEADER_2x05_PARALLEL, U1 MS5611-01BA

Commit message: resave
Parts:
- R1, R2: value 5k -> 5k1
Changed lines of the file:
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@@
     (property "Sheetfile" "ALTIMET02.kicad_sch")
     (property "Sheetname" "")
+    (property "UST_ID" "")
     (property "ki_description" "2x05 2.54 mm pitch header, 2 pins next to each other are connected")
     (property "ki_keywords" "2x05, header, connector, pinheader")
@@
     (property "Sheetfile" "ALTIMET02.kicad_sch")
     (property "Sheetname" "")
+    (property "UST_ID" "")
     (property "ki_description" "2x02 2.54 mm pitch header, 2 pins next to each other are connected")
     (property "ki_keywords" "2x02, header, connector, pinheader")
@@
     (property "Sheetfile" "ALTIMET02.kicad_sch")
     (property "Sheetname" "")
+    (property "UST_ID" "")
     (property "ki_description" "Mounting Hole with connection")
     (property "ki_keywords" "mounting hole")
@@
     (property "Sheetfile" "ALTIMET02.kicad_sch")
     (property "Sheetname" "")
+    (property "UST_ID" "")
     (property "ki_description" "Mounting Hole with connection")
     (property "ki_keywords" "mounting hole")
@@
     (property "Sheetfile" "ALTIMET02.kicad_sch")
     (property "Sheetname" "")
+    (property "UST_ID" "")
     (property "ki_description" "2x03 2.54 mm pitch header, 2 pins next to each other are connected")
     (property "ki_keywords" "2x03, header, connector, pinheader")
@@
     (property "Sheetfile" "ALTIMET02.kicad_sch")
     (property "Sheetname" "")
+    (property "UST_ID" "")
     (property "ki_description" "3-pole Solder Jumper, pins 1+2 closed/bridged")
     (property "ki_keywords" "Solder Jumper SPDT")
@@
     (property "Sheetfile" "ALTIMET02.kicad_sch")
     (property "Sheetname" "")
+    (property "UST_ID" "")
     (property "ki_description" "Mounting Hole with connection")
     (property "ki_keywords" "mounting hole")
@@
     (property "Sheetfile" "ALTIMET02.kicad_sch")
     (property "Sheetname" "")
+    (property "UST_ID" "")
     (property "ki_description" "Mounting Hole with connection")
     (property "ki_keywords" "mounting hole")
@@
     (property "Sheetfile" "ALTIMET02.kicad_sch")
     (property "Sheetname" "")
+    (property "UST_ID" "5fa0fc3e12875025b3977997")
     (property "ki_description" "Resistor")
     (property "ki_keywords" "R res resistor")
@@
         (effects (font (size 1 1) (thickness 0.15)) (justify mirror))
     )
-    (fp_text value "5k" (at 0 1.524) (layer "B.Fab")
+    (fp_text value "5k1" (at 0 1.524) (layer "B.Fab")
         (effects (font (size 1 1) (thickness 0.15)) (justify mirror))
     )
@@
     (property "Sheetfile" "ALTIMET02.kicad_sch")
     (property "Sheetname" "")
+    (property "UST_ID" "5c70984712875079b91f8b4c")
     (property "ki_description" "Unpolarized capacitor")
     (property "ki_keywords" "cap capacitor")
@@
     (property "Sheetfile" "ALTIMET02.kicad_sch")
     (property "Sheetname" "")
+    (property "UST_ID" "650b36b0462c6d9e720543f4")
     (property "ki_description" "Barometric pressure sensor, 10cm resolution, 10 to 1200 mbar, I2C and SPI interface up to 20MHz, LGA-8")
     (property "ki_keywords" "pressure SPI I2C")
@@
     (property "Sheetfile" "ALTIMET02.kicad_sch")
     (property "Sheetname" "")
+    (property "UST_ID" "650b35ab462c6d9e720543d0")
     (property "ki_description" "Zener diode")
     (property "ki_keywords" "diode")
@@
     (property "Sheetfile" "ALTIMET02.kicad_sch")
     (property "Sheetname" "")
+    (property "UST_ID" "")
     (property "ki_description" "Fiducial Marker")
     (property "ki_keywords" "fiducial marker")
@@
     (property "Sheetfile" "ALTIMET02.kicad_sch")
     (property "Sheetname" "")
+    (property "UST_ID" "5fa0fc3e12875025b3977997")
     (property "ki_description" "Resistor")
     (property "ki_keywords" "R res resistor")
@@
         (effects (font (size 1 1) (thickness 0.15)) (justify mirror))
     )
-    (fp_text value "5k" (at 1.153 -4.148928) (layer "B.Fab")
+    (fp_text value "5k1" (at 1.153 -4.148928) (layer "B.Fab")
         (effects (font (size 1 1) (thickness 0.15)) (justify mirror))
     )
@@
     (property "Sheetfile" "ALTIMET02.kicad_sch")
     (property "Sheetname" "")
+    (property "UST_ID" "")
     (property "ki_description" "Fiducial Marker")
     (property "ki_keywords" "fiducial marker")
@@
     (property "Sheetfile" "ALTIMET02.kicad_sch")
     (property "Sheetname" "")
+    (property "UST_ID" "5c70984712875079b91f8b53")
     (property "ki_description" "Unpolarized capacitor")
     (property "ki_keywords" "cap capacitor")
@@
     (property "Sheetfile" "ALTIMET02.kicad_sch")
     (property "Sheetname" "")
+    (property "UST_ID" "")
     (property "ki_description" "3-pole Solder Jumper, pins 1+2 closed/bridged")
     (property "ki_keywords" "Solder Jumper SPDT")

Commit message: Upravy a kontrola pred vyrobou
Parts:
- U1: footprint Package_LGA:LGA-8_3x5mm_P1.25mm -> Mlab_IO:MS5611-01BA03
- moved C2 0.29 mm to (136.7, 108.6)
- moved R2 0.22 mm to (134.4, 104.3)
Routing:
- net GND: track 0.00 -> 1.28 mm
- net VDD: track 34.3 -> 33.7 mm
Other:
- rule pad_to_mask_clearance: 0 -> 0.2
Changed lines of the file:
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@@
   )
   (setup
-    (pad_to_mask_clearance 0)
+    (stackup
+      (layer "F.SilkS" (type "Top Silk Screen"))
+      (layer "F.Paste" (type "Top Solder Paste"))
+      (layer "F.Mask" (type "Top Solder Mask") (thickness 0.01))
+      (layer "F.Cu" (type "copper") (thickness 0.035))
+      (layer "dielectric 1" (type "core") (thickness 1.51) (material "FR4") (epsilon_r 4.5) (loss_tangent 0.02))
+      (layer "B.Cu" (type "copper") (thickness 0.035))
+      (layer "B.Mask" (type "Bottom Solder Mask") (thickness 0.01))
+      (layer "B.Paste" (type "Bottom Solder Paste"))
+      (layer "B.SilkS" (type "Bottom Silk Screen"))
+      (copper_finish "None")
+      (dielectric_constraints no)
+    )
+    (pad_to_mask_clearance 0.2)
     (pcbplotparams
       (layerselection 0x00010fc_ffffffff)
@@
     (pad "1" thru_hole circle (at 0 0) (size 6 6) (drill 3) (layers "*.Cu" "*.Mask")
       (net 6 "GND") (pinfunction "1") (pintype "input") (clearance 1) (zone_connect 2))
-    (model "${MLAB}/src/3d/mechanical/m3_komplet.step"
+    (model "${MLAB_3DMODEL_DIR}/DIN_912-M3x10.stp"
       (offset (xyz 0 0 0))
       (scale (xyz 1 1 1))
-      (rotate (xyz 0 0 0))
+      (rotate (xyz 0 -90 0))
     )
   )
@@
     (pad "1" thru_hole circle (at 0 0) (size 6 6) (drill 3) (layers "*.Cu" "*.Mask")
       (net 6 "GND") (pinfunction "1") (pintype "input") (clearance 1) (zone_connect 2))
-    (model "${MLAB}/src/3d/mechanical/m3_komplet.step"
+    (model "${MLAB_3DMODEL_DIR}/DIN_912-M3x10.stp"
       (offset (xyz 0 0 0))
       (scale (xyz 1 1 1))
-      (rotate (xyz 0 0 0))
+      (rotate (xyz 0 -90 0))
     )
   )
@@
     (pad "1" thru_hole circle (at 0 0) (size 6 6) (drill 3) (layers "*.Cu" "*.Mask")
       (net 6 "GND") (pinfunction "1") (pintype "input") (clearance 1) (zone_connect 2))
-    (model "${MLAB}/src/3d/mechanical/m3_komplet.step"
+    (model "${MLAB_3DMODEL_DIR}/DIN_912-M3x10.stp"
       (offset (xyz 0 0 0))
       (scale (xyz 1 1 1))
-      (rotate (xyz 0 0 0))
+      (rotate (xyz 0 -90 0))
     )
   )
@@
     (pad "1" thru_hole circle (at 0 0) (size 6 6) (drill 3) (layers "*.Cu" "*.Mask")
       (net 6 "GND") (pinfunction "1") (pintype "input") (clearance 1) (zone_connect 2))
-    (model "${MLAB}/src/3d/mechanical/m3_komplet.step"
+    (model "${MLAB_3DMODEL_DIR}/DIN_912-M3x10.stp"
       (offset (xyz 0 0 0))
       (scale (xyz 1 1 1))
-      (rotate (xyz 0 0 0))
+      (rotate (xyz 0 -90 0))
     )
   )
@@
     (property "ki_keywords" "R res resistor")
     (attr smd)
-    (fp_text reference "R1" (at 2.54 0) (layer "B.SilkS")
+    (fp_text reference "R1" (at 2.54 -0.414) (layer "B.SilkS")
         (effects (font (size 1 1) (thickness 0.15)) (justify mirror))
     )
@@
   )
   (footprint "Capacitor_SMD:C_0805_2012Metric" (layer "B.Cu")
-    (at 136.3626 108.612 90)
+    (at 136.652 108.612 90)
     (descr "Capacitor SMD 0805 (2012 Metric), square (rectangular) end terminal, IPC_7351 nominal, (Body size source: IPC-SM-782 page 76, https://www.pcb-3d.com/wordpress/wp-content/uploads/ipc-sm-782a_amendment_1_and_2.pdf, https://docs.google.com/spreadsheets/d/1BsfQQcO9C6DZCsRaXUlFlo91Tg2WpOkGARC1WS5S8t0/edit?usp=sharing), generated with kicad-footprint-generator")
     (tags "capacitor")
@@
     )
   )
-  (footprint "Package_LGA:LGA-8_3x5mm_P1.25mm" (layer "B.Cu")
+  (footprint "Mlab_IO:MS5611-01BA03" (layer "B.Cu")
     (at 129.9464 108.1224 90)
     (descr "LGA-8")
@@
     (fp_line (start 1.5 2.5) (end 1.5 -2.5)
       (stroke (width 0.1) (type solid)) (layer "B.Fab"))
-    (pad "1" smd rect (at -1.075 1.875 90) (size 0.95 0.55) (layers "B.Cu" "B.Paste" "B.Mask")
+    (pad "1" smd rect (at -1.1 1.875 90) (size 1.1 0.6) (layers "B.Cu" "B.Paste" "B.Mask")
       (net 1 "VDD") (pinfunction "VDD") (pintype "power_in"))
-    (pad "2" smd rect (at -1.075 0.625 90) (size 0.95 0.55) (layers "B.Cu" "B.Paste" "B.Mask")
+    (pad "2" smd rect (at -1.1 0.625 90) (size 1.1 0.6) (layers "B.Cu" "B.Paste" "B.Mask")
       (net 5 "/PS") (pinfunction "PS") (pintype "input"))
-    (pad "3" smd rect (at -1.075 -0.625 90) (size 0.95 0.55) (layers "B.Cu" "B.Paste" "B.Mask")
+    (pad "3" smd rect (at -1.1 -0.625 90) (size 1.1 0.6) (layers "B.Cu" "B.Paste" "B.Mask")
       (net 6 "GND") (pinfunction "GND") (pintype "power_in"))
-    (pad "4" smd rect (at -1.075 -1.875 90) (size 0.95 0.55) (layers "B.Cu" "B.Paste" "B.Mask")
+    (pad "4" smd rect (at -1.1 -1.875 90) (size 1.1 0.6) (layers "B.Cu" "B.Paste" "B.Mask")
       (net 4 "CS{slash}A") (pinfunction "CSB") (pintype "input"))
-    (pad "5" smd rect (at 1.075 -1.875 90) (size 0.95 0.55) (layers "B.Cu" "B.Paste" "B.Mask")
+    (pad "5" smd rect (at 1.1 -1.875 90) (size 1.1 0.6) (layers "B.Cu" "B.Paste" "B.Mask")
       (net 4 "CS{slash}A") (pinfunction "CSB") (pintype "input"))
-    (pad "6" smd rect (at 1.075 -0.625 90) (size 0.95 0.55) (layers "B.Cu" "B.Paste" "B.Mask")
+    (pad "6" smd rect (at 1.1 -0.625 90) (size 1.1 0.6) (layers "B.Cu" "B.Paste" "B.Mask")
       (net 3 "MISO") (pinfunction "SDO") (pintype "output"))
-    (pad "7" smd rect (at 1.075 0.625 90) (size 0.95 0.55) (layers "B.Cu" "B.Paste" "B.Mask")
+    (pad "7" smd rect (at 1.1 0.625 90) (size 1.1 0.6) (layers "B.Cu" "B.Paste" "B.Mask")
       (net 2 "MOSI{slash}SDA") (pinfunction "SDI/SDA") (pintype "bidirectional"))
-    (pad "8" smd rect (at 1.075 1.875 90) (size 0.95 0.55) (layers "B.Cu" "B.Paste" "B.Mask")
+    (pad "8" smd rect (at 1.1 1.875 90) (size 1.1 0.6) (layers "B.Cu" "B.Paste" "B.Mask")
       (net 7 "SCLK") (pinfunction "SCLK") (pintype "input"))
     (model "${KICAD6_3DMODEL_DIR}/Package_LGA.3dshapes/LGA-8_3x5mm_P1.25mm.wrl"
@@
   )
   (footprint "Resistor_SMD:R_0805_2012Metric" (layer "B.Cu")
-    (at 134.5875 104.3 180)
+    (at 134.366 104.3 180)
     (descr "Resistor SMD 0805 (2012 Metric), square (rectangular) end terminal, IPC_7351 nominal, (Body size source: IPC-SM-782 page 72, https://www.pcb-3d.com/wordpress/wp-content/uploads/ipc-sm-782a_amendment_1_and_2.pdf), generated with kicad-footprint-generator")
     (tags "resistor")
@@
   (gr_line (start 152.146 96.774) (end 152.146 116.586)
     (stroke (width 0.127) (type solid)) (layer "Edge.Cuts"))
-  (gr_text "ALTIMET02A" (at 146.2 106.68) (layer "F.Cu")
-    (effects (font (size 1 1) (thickness 0.15)))
-  )
-  (gr_text "MLAB.cz" (at 116.84 106.68) (layer "F.Cu")
-    (effects (font (size 1 1) (thickness 0.15)))
-  )
   (gr_text "MLAB.cz" (at 147.32 106.68) (layer "B.Cu")
     (effects (font (size 1 1) (thickness 0.15)) (justify mirror))
@@
   (segment (start 131.8214 112.4214) (end 131.8214 113.4474) (width 0.508) (layer "B.Cu") (net 1))
   (segment (start 136.4 101.856) (end 136.4 104.392) (width 0.508) (layer "B.Cu") (net 1))
-  (segment (start 138.684 108.43) (end 138.712 108.458) (width 0.508) (layer "B.Cu") (net 1))
   (segment (start 138.712 109.562) (end 136.3626 109.562) (width 0.508) (layer "B.Cu") (net 1))
   (segment (start 131.824 109.2) (end 131.8214 109.1974) (width 0.508) (layer "B.Cu") (net 1))
@@
   (segment (start 131.8214 109.1974) (end 131.8214 112.3786) (width 0.508) (layer "B.Cu") (net 1))
   (segment (start 138.712 111.732) (end 138.684 111.76) (width 0.508) (layer "B.Cu") (net 1))
-  (segment (start 132 113.626) (end 132 113.8) (width 0.2) (layer "B.Cu") (net 1))
   (segment (start 138.684 111.76) (end 138.684 114.3) (width 0.508) (layer "B.Cu") (net 1))
-  (segment (start 134.1066 109.592) (end 134.0766 109.562) (width 0.508) (layer "B.Cu") (net 1))
   (segment (start 138.712 108.458) (end 138.712 111.732) (width 0.508) (layer "B.Cu") (net 1))
   (segment (start 131.8214 113.4474) (end 132 113.626) (width 0.508) (layer "B.Cu") (net 1))
   (segment (start 131.8 112.4) (end 131.8214 112.4214) (width 0.508) (layer "B.Cu") (net 1))
   (segment (start 136.398 99.314) (end 136.398 101.854) (width 0.508) (layer "B.Cu") (net 1))
-  (segment (start 131.826 108.97) (end 131.826 109.22) (width 0.25) (layer "B.Cu") (net 1))
   (segment (start 131.8214 112.3786) (end 131.8 112.4) (width 0.508) (layer "B.Cu") (net 1))
-  (segment (start 134.0766 109.562) (end 133.975 109.6636) (width 0.508) (layer "B.Cu") (net 1))
   (segment (start 134.0766 109.562) (end 133.7146 109.2) (width 0.508) (layer "B.Cu") (net 1))
   (segment (start 133.858 103.9895) (end 133.4535 104.394) (width 0.4) (layer "B.Cu") (net 2))
@@
   (via (at 127.254 112.776) (size 0.8) (drill 0.4) (layers "F.Cu" "B.Cu") (free) (net 6))
   (via (at 135.382 106.426) (size 0.8) (drill 0.4) (layers "F.Cu" "B.Cu") (free) (net 6))
-  (via (at 129.9 108.1) (size 0.8) (drill 0.4) (layers "F.Cu" "B.Cu") (free) (net 6))
+  (via (at 129.286 110.49) (size 0.8) (drill 0.4) (layers "F.Cu" "B.Cu") (free) (net 6))
   (via (at 127.254 113.792) (size 0.8) (drill 0.4) (layers "F.Cu" "B.Cu") (free) (net 6))
+  (segment (start 129.286 109.2578) (end 129.3214 109.2224) (width 0.25) (layer "B.Cu") (net 6))
+  (segment (start 129.286 110.49) (end 129.286 109.2578) (width 0.25) (layer "B.Cu") (net 6))
   (segment (start 138.938 103.9895) (end 138.938 105.162) (width 0.4) (layer "B.Cu") (net 7))
   (segment (start 138.938 101.854) (end 138.938 103.9895) (width 0.4) (layer "B.Cu") (net 7))
@@
       )
     )
+  )
+  (zone (net 0) (net_name "") (layer "B.Cu") (hatch edge 0.5)
+    (connect_pads (clearance 0))
+    (min_thickness 0.25) (filled_areas_thickness no)
+    (keepout (tracks allowed) (vias allowed) (pads allowed) (copperpour not_allowed) (footprints allowed))
+    (fill (thermal_gap 0.5) (thermal_bridge_width 0.5))
+    (polygon
+      (pts
+        (xy 127.762 106.426)
+        (xy 132.334 106.426)
+        (xy 132.334 109.728)
+        (xy 127.762 109.728)
+      )
+    )
